Commit message: add walls in version 4

File: my_ur/urdf/model1.urdf (robot description, URDF)
Before this commit: robot my_ur3e, 13 links, 12 joints
Links:
- added link wall_front, mass 200.0; collision box size=0.1 1 1
- added link wall_left, mass 200.0; collision box size=1 0.1 1
- added link wall_right, mass 200.0; collision box size=1 0.1 1
- link blob: geometry collision box size=1.0 1.0 1.0; visual box size=1 1 1
Joints:
- added joint blob-wall_front: type fixed, parent blob, child wall_front, origin xyz=-0.50 0.0 1.0 rpy=0.0 0.0 0.0
- added joint blob-wall_left: type fixed, parent blob, child wall_left, origin xyz=0.0 0.50 1. rpy=0.0 0.0 0.0
- added joint blob-wall_right: type fixed, parent blob, child wall_right, origin xyz=0.0 -0.5 1 rpy=0.0 0.0 0.0
